Commit message: Edit microsteps to 1600

File: src/stepperbot_description/urdf/stepperbot.urdf.xacro (robot description, xacro)
@@ -47,5 +47,5 @@
     <origin xyz="0 0 ${motor_length}" rpy="0 0 0"/>
     <axis xyz="0 0 1"/>
-    <limit lower="-6.283" upper="6.283" velocity="10" effort="1"/>
+    <limit lower="-6.283" upper="6.283" velocity="100" effort="1"/>
   </joint>
   <!-- Motor 2 -->
@@ -76,5 +76,5 @@
     <origin xyz="0 0 ${motor_length}" rpy="0 0 0"/>
     <axis xyz="0 0 1"/>
-    <limit lower="-6.283" upper="6.283" velocity="10" effort="1"/>
+    <limit lower="-6.283" upper="6.283" velocity="100" effort="1"/>
   </joint>
 </robot>
